Commit message: Add files via upload

File: src/my_robot/urdf/my_robot.xacro (robot description, xacro)
@@ -42,5 +42,4 @@
     <visual name="back_caster_visual">
       <origin xyz="-0.15 0 -0.075" rpy="0 0 0"/>
-<<<<<<< HEAD
       <geometry>
         <sphere radius="0.075"/>
@@ -61,14 +60,8 @@
         <sphere radius="0.075"/>
       </geometry>
-=======
-      <geometry>
-        <sphere radius="0.075"/>
-      </geometry>
->>>>>>> d8cc4a8626a1684f31ceb1ddc6028cf524a822ba
       <material name="">
         <color rgba="1 1 0 1"/>
       </material>
     </visual>
-<<<<<<< HEAD
   </link>
   <link name="left_wheel">
@@ -202,47 +195,4 @@
       </geometry>
     </visual>
-=======
-    <collision name="front_caster_collision">
-      <origin xyz="0.15 0 -0.075" rpy="0 0 0"/>
-      <geometry>
-        <sphere radius="0.0749"/>
-      </geometry>
-    </collision>
-    <visual name="front_caster_visual">
-      <origin xyz="0.15 0 -0.075" rpy="0 0 0"/>
-      <geometry>
-        <sphere radius="0.075"/>
-      </geometry>
-      <material name="">
-        <color rgba="1 1 0 1"/>
-      </material>
-    </visual>
-  </link>
-  <link name="left_wheel">
-    <inertial>
-      <mass value="5.0"/>
-      <origin xyz="0 0 0" rpy="0 0 0"/>
-      <inertia
-          ixx="0.1" ixy="0" ixz="0"
-          iyy="0.1" iyz="0"
-          izz="0.1"
-      />
-    </inertial>
-    <collision name="left_wheel_collision">
-      <origin xyz="0 0 0" rpy="0 1.5707 1.5707"/>
-      <geometry>
-        <cylinder radius="0.15" length="0.05"/>
-      </geometry>
-    </collision>
-    <visual name="left_wheel_visual">
-      <origin xyz="0 0 0" rpy="0 1.5707 1.5707"/>
-      <geometry>
-        <cylinder radius="0.15" length="0.05"/>
-      </geometry>
-      <material name="Green">
-        <color rgba="0 1 0 1"/>
-      </material>
-    </visual>
->>>>>>> d8cc4a8626a1684f31ceb1ddc6028cf524a822ba
   </link>
   <!-- HOKUYO LIDAR JOINT -->
@@ -253,119 +203,4 @@
     <axis xyz="0 1 0"/>
   </joint>
-<<<<<<< HEAD
-=======
-  <!-- LEFT WHEEL JOINT -->
-  <joint type="continuous" name="left_wheel_hinge">
-    <origin xyz="0 0.2 0" rpy="0 0 0"/>
-    <child link="left_wheel"/>
-    <parent link="chassis"/>
-    <axis xyz="0 1 0"/>
-    <limit effort="10000" velocity="1000"/>
-    <dynamics damping="1.0" friction="1.0"/>
-  </joint>
-  <!-- RIGHT WHEEL LINK -->
-  <link name="right_wheel">
-    <inertial>
-      <mass value="5.0"/>
-      <origin xyz="0 0 0" rpy="0 0 0"/>
-      <inertia
-          ixx="0.1" ixy="0" ixz="0"
-          iyy="0.1" iyz="0"
-          izz="0.1"
-      />
-    </inertial>
-    <collision name="right_wheel_collision">
-      <origin xyz="0 0 0" rpy="0 1.5708 1.5708"/>
-      <geometry>
-        <!-- Wheel radius remains 0.15 -->
-        <cylinder radius="0.15" length="0.05"/>
-      </geometry>
-    </collision>
-    <visual name="right_wheel_visual">
-      <origin xyz="0 0 0" rpy="0 1.5707 1.5707"/>
-      <geometry>
-        <cylinder radius="0.15" length="0.05"/>
-      </geometry>
-      <!-- Green wheels -->
-      <material name="Green">
-        <color rgba="0 1 0 1"/>
-      </material>
-    </visual>
-  </link>
-  <!-- RIGHT WHEEL JOINT -->
-  <joint type="continuous" name="right_wheel_hinge">
-    <origin xyz="0 -0.2 0" rpy="0 0 0"/>
-    <child link="right_wheel"/>
-    <parent link="chassis"/>
-    <axis xyz="0 1 0"/>
-    <limit effort="10000" velocity="1000"/>
-    <dynamics damping="1.0" friction="1.0"/>
-  </joint>
-  <!-- CAMERA LINK -->
-  <link name="camera">
-    <inertial>
-      <mass value="0.1"/>
-      <origin xyz="0 0 0" rpy="0 0 0"/>
-      <inertia
-          ixx="1e-6" ixy="0" ixz="0"
-          iyy="1e-6" iyz="0"
-          izz="1e-6"
-      />
-    </inertial>
-    <collision>
-      <origin xyz="0 0 0" rpy="0 0 0"/>
-      <geometry>
-        <box size="0.05 0.05 0.05"/>
-      </geometry>
-    </collision>
-    <visual>
-      <origin xyz="0 0 0" rpy="0 0 0"/>
-      <geometry>
-        <box size="0.05 0.05 0.05"/>
-      </geometry>
-      <material name="Red">
-        <color rgba="1 0 0 1"/>
-      </material>
-    </visual>
-  </link>
-  <!-- CAMERA JOINT -->
-  <joint name="camera_joint" type="fixed">
-    <origin xyz="0.25 0 0" rpy="0 0 0"/>
-    <parent link="chassis"/>
-    <child link="camera"/>
-    <axis xyz="0 1 0"/>
-  </joint>
-  <!-- HOKUYO LIDAR LINK -->
-  <link name="hokuyo">
-    <inertial>
-      <mass value="1e-5"/>
-      <origin xyz="0 0 0" rpy="0 0 0"/>
-      <inertia
-          ixx="1e-6" ixy="0" ixz="0"
-          iyy="1e-6" iyz="0"
-          izz="1e-6"
-      />
-    </inertial>
-    <collision>
-      <origin xyz="0 0 0" rpy="0 0 0"/>
-      <geometry>
-        <box size="0.1 0.1 0.1"/>
-      </geometry>
-    </collision>
-    <visual>
-      <origin xyz="0 0 0" rpy="0 0 0"/>
-      <geometry>
-        <mesh filename="package://my_robot/meshes/hokuyo.dae"/>
-      </geometry>
-    </visual>
-  </link>
-  <!-- HOKUYO LIDAR JOINT -->
-  <joint name="hokuyo_joint" type="fixed">
-    <origin xyz="0.2 0 0.1" rpy="0 0 0"/>
-    <parent link="chassis"/>
-    <child link="hokuyo"/>
-    <axis xyz="0 1 0"/>
-  </joint>
->>>>>>> d8cc4a8626a1684f31ceb1ddc6028cf524a822ba
   <!-- Gazebo color Chasis -->
   <gazebo reference="chassis">
